Commit message: asdf

File: autodex/planner/src/curobo/content/assets/robot/inspire_description/xarm_inspire.urdf (robot description, URDF)
Before this commit: robot combined_robot, 22 links, 21 joints
Joints:
- joint joint1: origin xyz=0 0 0.267 rpy=0 0 0 -> xyz=-0.001549459761 0.0003137374879 0.2656630874 rpy=-0.002122362144 -0.002407404361 2.55469422e-06
- joint joint2: origin xyz=0 0 0 rpy=-1.5708 0 0 -> xyz=0.0001424681977 -4.629010846e-07 -5.750245766e-11 rpy=-1.570928454 0.002410640009 -0.003248984925
- joint joint3: origin xyz=0.0535 -0.2845 0 rpy=0 0 0 -> xyz=0.05299152806 -0.2844330966 5.917066301e-05 rpy=-0.001330370083 -0.001908135135 -3.037097713e-06
- joint joint4: origin xyz=0.0775 0.3425 0 rpy=-1.5708 0 0 -> xyz=0.07818619162 0.3414653838 -0.0005268830573 rpy=-1.57233882 -0.001340431976 -0.002912688535
- joint joint5: origin xyz=0 0 0 rpy=1.5708 0 0 -> xyz=-0.0003658483038 -0.002068420639 -3.251171802e-05 rpy=1.586496472 -0.002846868243 -0.006097148173
- joint joint6: origin xyz=0.076 0.097 0 rpy=-1.5708 0 0 -> xyz=0.07646542042 0.0960168317 -0.0008099220577 rpy=-1.581605673 0.005988837685 -0.000228099816

File: src/grasp_generation/BODex/src/curobo/content/assets/robot/allegro_description/xarm_allegro.urdf (robot description, URDF)
Before this commit: robot combined_robot, 30 links, 29 joints
Joints:
- joint joint1: origin xyz=0 0 0.267 rpy=0 0 0 -> xyz=-0.001549459761 0.0003137374879 0.2656630874 rpy=-0.002122362144 -0.002407404361 2.55469422e-06
- joint joint2: origin xyz=0 0 0 rpy=-1.5708 0 0 -> xyz=0.0001424681977 -4.629010846e-07 -5.750245766e-11 rpy=-1.570928454 0.002410640009 -0.003248984925
- joint joint3: origin xyz=0.0535 -0.2845 0 rpy=0 0 0 -> xyz=0.05299152806 -0.2844330966 5.917066301e-05 rpy=-0.001330370083 -0.001908135135 -3.037097713e-06
- joint joint4: origin xyz=0.0775 0.3425 0 rpy=-1.5708 0 0 -> xyz=0.07818619162 0.3414653838 -0.0005268830573 rpy=-1.57233882 -0.001340431976 -0.002912688535
- joint joint5: origin xyz=0 0 0 rpy=1.5708 0 0 -> xyz=-0.0003658483038 -0.002068420639 -3.251171802e-05 rpy=1.586496472 -0.002846868243 -0.006097148173
- joint joint6: origin xyz=0.076 0.097 0 rpy=-1.5708 0 0 -> xyz=0.07646542042 0.0960168317 -0.0008099220577 rpy=-1.581605673 0.005988837685 -0.000228099816
